Commit message: Added noise file and default file

File: working_dir/catkin_ws/src/hector_quadrotor_noetic/hector_models/hector_sensors_description/urdf/sonar_sensor2.urdf.xacro (robot description, xacro)
@@ -55,5 +55,5 @@
         </ray>
         <plugin name="gazebo_ros_${name}_controller" filename="libhector_gazebo_ros_sonar.so">
-          <gaussianNoise>0.5</gaussianNoise>
+          <gaussianNoise>0.005</gaussianNoise>
           <topicName>${ros_topic}</topicName>
           <frameId>${name}_link</frameId>

File: working_dir/catkin_ws/src/hector_quadrotor_noetic/hector_models/hector_sensors_description/urdf/updated_sonar_sensor.urdf.xacro (robot description, xacro)
@@ -1,7 +1,7 @@
-<?xml version="1.0"?>
+<?xml version='1.0' encoding='UTF-8'?>
 <robot xmlns:xacro="http://ros.org/wiki/xacro">
   <xacro:macro name="sonar_sensor" params="name parent *origin ros_topic update_rate min_range max_range field_of_view ray_count">
     <joint name="${name}_joint" type="fixed">
-      <xacro:insert_block name="origin" />
+      <xacro:insert_block name="origin"/>
       <parent link="${parent}"/>
       <child link="${name}_link"/>
@@ -9,10 +9,10 @@
     <link name="${name}_link">
       <inertial>
-        <mass value="0.001" />
-        <origin xyz="0 0 0" rpy="0 0 0" />
-        <inertia ixx="0.000000017" ixy="0" ixz="0" iyy="0.000000017" iyz="0" izz="0.000000017" />
+        <mass value="0.001"/>
+        <origin xyz="0 0 0" rpy="0 0 0"/>
+        <inertia ixx="0.000000017" ixy="0" ixz="0" iyy="0.000000017" iyz="0" izz="0.000000017"/>
       </inertial>
       <visual>
-        <origin xyz="0 0 0" rpy="0 0 0" />
+        <origin xyz="0 0 0" rpy="0 0 0"/>
         <geometry>
           <!--<box size="0.01 0.01 0.01" /> -->
@@ -21,7 +21,7 @@
       </visual>
       <collision>
-        <origin xyz="0 0 0" rpy="0 0 0" />
+        <origin xyz="0 0 0" rpy="0 0 0"/>
         <geometry>
-          <box size="0.01 0.01 0.01" />
+          <box size="0.01 0.01 0.01"/>
         </geometry>
       </collision>
@@ -55,5 +55,5 @@
         </ray>
         <plugin name="gazebo_ros_${name}_controller" filename="libhector_gazebo_ros_sonar.so">
-          <gaussianNoise>0.5</gaussianNoise>
+          <gaussianNoise>2.0</gaussianNoise>
           <topicName>${ros_topic}</topicName>
           <frameId>${name}_link</frameId>

File: working_dir/catkin_ws/src/hector_quadrotor_noetic/hector_quadrotor/hector_quadrotor_description/urdf/quadrotor_downward_cam.urdf.xacro (robot description, xacro)
@@ -9,5 +9,34 @@
     <xacro:include filename="$(find hector_sensors_description)/urdf/generic_camera.urdf.xacro" />
     <xacro:generic_camera name="downward_cam" parent="base_link" ros_topic="camera/image" cam_info_topic="camera/camera_info" update_rate="20" res_x="640" res_y="480" image_format="L8" hfov="100">
-      <origin xyz="0.4 0.0 -0.0" rpy="0 ${M_PI/2} 0"/>
-    </xacro:generic_camera>
+      <origin xyz="0.0 0.0 0.0" rpy="0 ${M_PI/2} 0"/>
+<!--    </xacro:generic_camera>-->
+<!--    <gazebo reference="base_link">-->
+<!--    <material>Gazebo/Blue</material>-->
+<!--    <sensor name="camera" type="camera">-->
+<!--        <pose> 0 0 0 0 ${M_PI/2} 0 </pose>-->
+<!--        <visualize>true</visualize>-->
+<!--        <update_rate>30</update_rate>-->
+<!--        <camera>-->
+<!--            <horizontal_fov>2</horizontal_fov>-->
+<!--            <image>-->
+<!--                <format>R8G8B8</format>-->
+<!--                <width>640</width>-->
+<!--                <height>480</height>-->
+<!--            </image>-->
+<!--            <clip>-->
+<!--                <near>0.05</near>-->
+<!--                <far>8.00</far>-->
+<!--            </clip>-->
+<!--            <noise>-->
+<!--                <type>gaussian</type>-->
+<!--                <mean>0.0</mean>-->
+<!--                <stddev>0.07</stddev>-->
+<!--            </noise>-->
+<!--        </camera>-->
+<!--        <plugin name="camera_controller" filename="libgazebo_ros_camera.so">-->
+<!--            <frame_name>camera_optical_link</frame_name>-->
+<!--            <cameraName>camera</cameraName>-->
+<!--        </plugin>-->
+<!--    </sensor>-->
+<!--</gazebo>-->
 </robot>

File: working_dir/catkin_ws/src/hector_quadrotor_noetic/hector_quadrotor/hector_quadrotor_gazebo/urdf/noisy_quadrotor_sensors.gazebo.xacro (robot description, xacro)
@@ -45,7 +45,7 @@
             <referenceAltitude>0.0</referenceAltitude>
             <drift>0.0 0.0 0.0</drift>
-            <gaussianNoise>0.5 0.5 0.5</gaussianNoise>
+            <gaussianNoise>0.021 0.021 0.021</gaussianNoise>
             <velocityDrift>0 0 0</velocityDrift>
-            <velocityGaussianNoise>0.3 0.3 0.3</velocityGaussianNoise>
+            <velocityGaussianNoise>0.05 0.05 0.05</velocityGaussianNoise>
           </plugin>
           <plugin name="quadrotor_groundtruth_sim" filename="libgazebo_ros_p3d.so">

File: working_dir/catkin_ws/src/hector_quadrotor_noetic/hector_quadrotor/hector_quadrotor_gazebo/urdf/quadrotor_sensors2.gazebo.xacro (robot description, xacro)
@@ -10,7 +10,7 @@
             <topicName>raw_imu</topicName>
             <rpyOffset>0 0 0</rpyOffset> <!-- deprecated -->
-            <gaussianNoise>0.1</gaussianNoise>  <!-- deprecated -->
+            <gaussianNoise>0</gaussianNoise>  <!-- deprecated -->
             <accelDrift>0.0 0.0 0.0</accelDrift>
-            <accelGaussianNoise>10.0 10.0 10.0</accelGaussianNoise>
+            <accelGaussianNoise>0.0 0.0 0.0</accelGaussianNoise>
             <rateDrift>0.0 0.0 0.0</rateDrift>
             <rateGaussianNoise>0.0 0.0 0.0</rateGaussianNoise>
@@ -45,7 +45,7 @@
             <referenceAltitude>0.0</referenceAltitude>
             <drift>0.0 0.0 0.0</drift>
-            <gaussianNoise>0.5 0.5 0.5</gaussianNoise>
+            <gaussianNoise>0.00 0.00 0.00</gaussianNoise>
             <velocityDrift>0 0 0</velocityDrift>
-            <velocityGaussianNoise>0.3 0.3 0.3</velocityGaussianNoise>
+            <velocityGaussianNoise>0.00 0.00 0.00</velocityGaussianNoise>
           </plugin>
           <plugin name="quadrotor_groundtruth_sim" filename="libgazebo_ros_p3d.so">
