Commit message: Final change of parameters

File: working_dir/catkin_ws/src/hector_quadrotor_noetic/hector_models/hector_sensors_description/urdf/sonar_sensor.urdf.xacro (robot description, xacro)
@@ -1,7 +1,7 @@
-<?xml version="1.0"?>
+<?xml version='1.0' encoding='UTF-8'?>
 <robot xmlns:xacro="http://ros.org/wiki/xacro">
   <xacro:macro name="sonar_sensor" params="name parent *origin ros_topic update_rate min_range max_range field_of_view ray_count">
     <joint name="${name}_joint" type="fixed">
-      <xacro:insert_block name="origin" />
+      <xacro:insert_block name="origin"/>
       <parent link="${parent}"/>
       <child link="${name}_link"/>
@@ -9,10 +9,10 @@
     <link name="${name}_link">
       <inertial>
-        <mass value="0.001" />
-        <origin xyz="0 0 0" rpy="0 0 0" />
-        <inertia ixx="0.000000017" ixy="0" ixz="0" iyy="0.000000017" iyz="0" izz="0.000000017" />
+        <mass value="0.001"/>
+        <origin xyz="0 0 0" rpy="0 0 0"/>
+        <inertia ixx="0.000000017" ixy="0" ixz="0" iyy="0.000000017" iyz="0" izz="0.000000017"/>
       </inertial>
       <visual>
-        <origin xyz="0 0 0" rpy="0 0 0" />
+        <origin xyz="0 0 0" rpy="0 0 0"/>
         <geometry>
           <!--<box size="0.01 0.01 0.01" /> -->
@@ -21,7 +21,7 @@
       </visual>
       <collision>
-        <origin xyz="0 0 0" rpy="0 0 0" />
+        <origin xyz="0 0 0" rpy="0 0 0"/>
         <geometry>
-          <box size="0.01 0.01 0.01" />
+          <box size="0.01 0.01 0.01"/>
         </geometry>
       </collision>
@@ -55,5 +55,5 @@
         </ray>
         <plugin name="gazebo_ros_${name}_controller" filename="libhector_gazebo_ros_sonar.so">
-          <gaussianNoise>0.5</gaussianNoise>
+          <gaussianNoise>10.0</gaussianNoise>
           <topicName>${ros_topic}</topicName>
           <frameId>${name}_link</frameId>

File: working_dir/catkin_ws/src/hector_quadrotor_noetic/hector_quadrotor/hector_quadrotor_gazebo/urdf/quadrotor_sensors.gazebo.xacro (robot description, xacro)
@@ -1,60 +1,62 @@
-<?xml version="1.0"?>
+<?xml version='1.0' encoding='UTF-8'?>
 <robot xmlns:xacro="http://www.ros.org/wiki/xacro">
   <!-- Quadrotor Sensor Plugins -->
   <xacro:macro name="quadrotor_sensors">
-        <gazebo>
-          <plugin name="quadrotor_imu_sim" filename="libhector_gazebo_ros_imu.so">
-            <updateRate>10.0</updateRate>
-            <bodyName>base_link</bodyName>
-            <frameId>base_link</frameId>
-            <topicName>raw_imu</topicName>
-            <rpyOffset>0 0 0</rpyOffset> <!-- deprecated -->
-            <gaussianNoise>0.1</gaussianNoise>  <!-- deprecated -->
-            <accelDrift>0.0 0.0 0.0</accelDrift>
-            <accelGaussianNoise>10.0 10.0 10.0</accelGaussianNoise>
-            <rateDrift>0.0 0.0 0.0</rateDrift>
-            <rateGaussianNoise>0.0 0.0 0.0</rateGaussianNoise>
-          </plugin>
-          <plugin name="quadrotor_baro_sim" filename="libhector_gazebo_ros_baro.so">
-            <updateRate>10.0</updateRate>
-            <bodyName>base_link</bodyName>
-            <frameId>base_link</frameId>
-            <topicName>pressure_height</topicName>
-            <altimeterTopicName>altimeter</altimeterTopicName>
-            <offset>0</offset>
-            <drift>0.0</drift>
-            <gaussianNoise>0.0</gaussianNoise>
-          </plugin>
-          <plugin name="quadrotor_magnetic_sim" filename="libhector_gazebo_ros_magnetic.so">
-            <updateRate>10.0</updateRate>
-            <bodyName>base_link</bodyName>
-            <frameId>base_link</frameId>
-            <topicName>magnetic</topicName>
-            <offset>0 0 0</offset>
-            <drift>0.0 0.0 0.0</drift>
-            <gaussianNoise>1.3e-2 1.3e-2 1.3e-2</gaussianNoise>
-          </plugin>
-          <plugin name="quadrotor_gps_sim" filename="libhector_gazebo_ros_gps.so">
-            <updateRate>4.0</updateRate>
-            <bodyName>base_link</bodyName>
-            <frameId>base_link</frameId>
-            <topicName>fix</topicName>
-            <velocityTopicName>fix_velocity</velocityTopicName>
-            <referenceLatitude>49.860246</referenceLatitude>
-            <referenceLongitude>8.687077</referenceLongitude>
-            <referenceAltitude>0.0</referenceAltitude>
-            <drift>0.0 0.0 0.0</drift>
-            <gaussianNoise>0.5 0.5 0.5</gaussianNoise>
-            <velocityDrift>0 0 0</velocityDrift>
-            <velocityGaussianNoise>0.3 0.3 0.3</velocityGaussianNoise>
-          </plugin>
-          <plugin name="quadrotor_groundtruth_sim" filename="libgazebo_ros_p3d.so">
-            <updateRate>100.0</updateRate>
-            <bodyName>base_link</bodyName>
-            <topicName>ground_truth/state</topicName>
-            <gaussianNoise>0.0</gaussianNoise>
-            <frameName>world</frameName>
-          </plugin>
-        </gazebo>
+    <gazebo>
+      <plugin name="quadrotor_imu_sim" filename="libhector_gazebo_ros_imu.so">
+        <updateRate>10.0</updateRate>
+        <bodyName>base_link</bodyName>
+        <frameId>base_link</frameId>
+        <topicName>raw_imu</topicName>
+        <rpyOffset>0.0 0.0 0.0</rpyOffset>
+        <!-- deprecated -->
+        <gaussianNoise>10.5</gaussianNoise>
+        <!-- deprecated -->
+        <accelDrift>0.0 0.0 0.0</accelDrift>
+        <accelGaussianNoise>0.0 0.0 0.0</accelGaussianNoise>
+        <rateDrift>0.0 0.0 0.0</rateDrift>
+        <rateGaussianNoise>0.0 0.0 0.0</rateGaussianNoise>
+      </plugin>
+      <plugin name="quadrotor_baro_sim" filename="libhector_gazebo_ros_baro.so">
+        <updateRate>10.0</updateRate>
+        <bodyName>base_link</bodyName>
+        <frameId>base_link</frameId>
+        <topicName>pressure_height</topicName>
+        <altimeterTopicName>altimeter</altimeterTopicName>
+        <offset>0.0</offset>
+        <drift>0.0</drift>
+        <gaussianNoise>1.0</gaussianNoise>
+      </plugin>
+      <plugin name="quadrotor_magnetic_sim" filename="libhector_gazebo_ros_magnetic.so">
+        <updateRate>10.0</updateRate>
+        <bodyName>base_link</bodyName>
+        <frameId>base_link</frameId>
+        <topicName>magnetic</topicName>
+        <offset>0.0 0.0 0.0</offset>
+        <drift>0.0 0.0 0.0</drift>
+        <gaussianNoise>0.0 0.0 0.0</gaussianNoise>
+      </plugin>
+      <plugin name="quadrotor_gps_sim" filename="libhector_gazebo_ros_gps.so">
+        <updateRate>4.0</updateRate>
+        <bodyName>base_link</bodyName>
+        <frameId>base_link</frameId>
+        <topicName>fix</topicName>
+        <velocityTopicName>fix_velocity</velocityTopicName>
+        <referenceLatitude>49.860246</referenceLatitude>
+        <referenceLongitude>8.687077</referenceLongitude>
+        <referenceAltitude>0.0</referenceAltitude>
+        <drift>0.0 0.0 0.0</drift>
+        <gaussianNoise>20.0 20.0 20.0</gaussianNoise>
+        <velocityDrift>0.0 0.0 0.0</velocityDrift>
+        <velocityGaussianNoise>0.0 0.0 0.0</velocityGaussianNoise>
+      </plugin>
+      <plugin name="quadrotor_groundtruth_sim" filename="libgazebo_ros_p3d.so">
+        <updateRate>100.0</updateRate>
+        <bodyName>base_link</bodyName>
+        <topicName>ground_truth/state</topicName>
+        <gaussianNoise>0.0</gaussianNoise>
+        <frameName>world</frameName>
+      </plugin>
+    </gazebo>
   </xacro:macro>
 </robot>
